Commit message: examples with kinova and dinova added

File: pumafabrics/tamed_puma/config/urdfs/dingo_kinova.urdf (robot description, URDF)
Before this commit: robot dingo_kinova, 27 links, 26 joints
Links:
- removed link arm_orientation_helper_link
Joints:
- removed joint arm_orientation_helper_joint
- joint arm_tool_frame_joint: origin xyz=0 0 0.070 rpy=0 0 0 -> xyz=0 0 0.130 rpy=0 0 0

File: pumafabrics/tamed_puma/config/urdfs/dinova_lidar.urdf (robot description, URDF)
Before this commit: robot dingo_kinova, 27 links, 26 joints
Joints:
- joint arm_mount_joint: origin xyz=0 0 0 rpy=0 0 0 -> xyz=0 0 0.314 rpy=0 0 0
