Commit message: examples of dinova and kinova work, also with TamedPUMA and more collision links

File: pumafabrics/tamed_puma/config/urdfs/gen3lite.urdf (robot description, URDF)
Before this commit: robot dingo_kinova, 16 links, 15 joints
Joints:
- joint right_finger_bottom_joint: type revolute -> fixed
