Commit message: removed redundant urdf files

File: pumafabrics/tamed_puma/config/urdfs/gen3lite_1.urdf (robot description, URDF)
Before this commit: robot kinova, 15 links, 14 joints
Links:
- added link orientation_helper_link
- link arm_link: geometry collision mesh filename=meshes/kinova/arm_link.STL; visual mesh filename=meshes/kinova/arm_link.STL
- link forearm_link: geometry collision mesh filename=meshes/kinova/forearm_link.STL; visual mesh filename=meshes/kinova/forearm_link.STL
- link gripper_base_link: geometry collision mesh filename=meshes/kinova/gripper_base_link.STL; visual mesh filename=/meshes/kinova/gripper_base_link.STL
- link kinova_base_link: geometry collision mesh filename=meshes/kinova/base_link.STL; visual mesh filename=meshes/kinova/base_link.STL
- link left_finger_dist_link: geometry collision mesh filename=meshes/kinova/left_finger_dist_link.STL; visual mesh filename=meshes/kinova/left_finger_dist_link.STL
- link left_finger_prox_link: geometry collision mesh filename=meshes/kinova/left_finger_prox_link.STL; visual mesh filename=meshes/kinova/left_finger_prox_link.STL
- link lower_wrist_link: geometry collision mesh filename=meshes/kinova/lower_wrist_link.STL; visual mesh filename=meshes/kinova/lower_wrist_link.STL
- link right_finger_dist_link: geometry collision mesh filename=meshes/kinova/right_finger_dist_link.STL; visual mesh filename=meshes/kinova/right_finger_dist_link.STL
- link right_finger_prox_link: geometry collision mesh filename=meshes/kinova/right_finger_prox_link.STL; visual mesh filename=meshes/kinova/right_finger_prox_link.STL
- link shoulder_link: geometry collision mesh filename=meshes/kinova/shoulder_link.STL; visual mesh filename=meshes/kinova/shoulder_link.STL
- link upper_wrist_link: geometry collision mesh filename=meshes/kinova/upper_wrist_link.STL; visual mesh filename=meshes/kinova/upper_wrist_link.STL
Joints:
- added joint orientation_helper_joint: type fixed, parent dummy_link, child orientation_helper_link, origin xyz=0 0.1 0 rpy=0 0 0, axis 0 0 0
- joint right_finger_bottom_joint: type revolute -> fixed
- joint tool_frame_joint: origin xyz=0 0 0.07 rpy=0 0 0 -> xyz=0 0 0.130 rpy=0 0 0

File: pumafabrics/tamed_puma/config/urdfs/gen3lite_2.urdf (robot description, URDF)
Before this commit: robot kinova, 15 links, 14 joints
Links:
- added link orientation_helper_link
- link arm_link: geometry collision mesh filename=meshes/kinova/arm_link.STL; visual mesh filename=meshes/kinova/arm_link.STL
- link forearm_link: geometry collision mesh filename=meshes/kinova/forearm_link.STL; visual mesh filename=meshes/kinova/forearm_link.STL
- link gripper_base_link: geometry collision mesh filename=meshes/kinova/gripper_base_link.STL; visual mesh filename=meshes/kinova/gripper_base_link.STL
- link kinova_base_link: geometry collision mesh filename=meshes/kinova/base_link.STL; visual mesh filename=meshes/kinova/base_link.STL
- link left_finger_dist_link: geometry collision mesh filename=meshes/kinova/left_finger_dist_link.STL; visual mesh filename=meshes/kinova/left_finger_dist_link.STL
- link left_finger_prox_link: geometry collision mesh filename=meshes/kinova/left_finger_prox_link.STL; visual mesh filename=meshes/kinova/left_finger_prox_link.STL
- link lower_wrist_link: geometry collision mesh filename=meshes/kinova/lower_wrist_link.STL; visual mesh filename=meshes/kinova/lower_wrist_link.STL
- link right_finger_dist_link: geometry collision mesh filename=meshes/kinova/right_finger_dist_link.STL; visual mesh filename=meshes/kinova/right_finger_dist_link.STL
- link right_finger_prox_link: geometry collision mesh filename=meshes/kinova/right_finger_prox_link.STL; visual mesh filename=meshes/kinova/right_finger_prox_link.STL
- link shoulder_link: geometry collision mesh filename=meshes/kinova/shoulder_link.STL; visual mesh filename=meshes/kinova/shoulder_link.STL
- link upper_wrist_link: geometry collision mesh filename=meshes/kinova/upper_wrist_link.STL; visual mesh filename=meshes/kinova/upper_wrist_link.STL
Joints:
- added joint orientation_helper_joint: type fixed, parent dummy_link, child orientation_helper_link, origin xyz=0 0.1 0 rpy=0 0 0, axis 0 0 0
- joint right_finger_bottom_joint: type revolute -> fixed
- joint tool_frame_joint: origin xyz=0 0 0.07 rpy=0 0 0 -> xyz=0 0 0.130 rpy=0 0 0
